File: cad_design/paper.sch (KiCad schematic (older format))
At the start: 5 parts

Commit message: Segundo Commit
En este commit se presenta el diseño de la tarjeta impresa para la
adecuación de las señales de voltaje y corriente, para empezar la
implementación.
Parts:
- removed J?: Conn_01x02_Female, symbol Connector:Conn_01x02_Female
- removed U?: LM358, symbol Amplifier_Operational:LM358
- added C2: 0.1uF, Capacitor_SMD:C_1206_3216Metric_Pad1.42x1.75mm_HandSolder, symbol pspice:CAP
- added J1: Conn_01x02, Connector_Wire:SolderWirePad_1x02_P5.08mm_Drill1.5mm, symbol Connector_Generic:Conn_01x02
- added J2: Conn_01x03, Connector_Wire:SolderWirePad_1x04_P5.08mm_Drill1.5mm, symbol Connector_Generic:Conn_01x03
- added J3: Conn_01x06, Connector_PinSocket_2.54mm:PinSocket_1x06_P2.54mm_Vertical, symbol Connector_Generic:Conn_01x06
- added J4: Conn_01x08, Connector_PinSocket_2.54mm:PinSocket_1x08_P2.54mm_Vertical, symbol Connector_Generic:Conn_01x08
- added R3: 22k, Resistor_SMD:R_1206_3216Metric, symbol Device:R_US
- added R4: 3.3k, Resistor_SMD:R_1206_3216Metric, symbol Device:R_US
- added U1: LM358, Package_DIP:DIP-8_W7.62mm_SMDSocket_SmallPads, symbol Amplifier_Operational:LM358
- C1: renamed from C?; value CAP -> 0.1uF; footprint (none) -> Capacitor_SMD:C_1206_3216Metric_Pad1.42x1.75mm_HandSolder
- R1: renamed from R?; value R_US -> 22k; footprint (none) -> Resistor_SMD:R_1206_3216Metric
- R2: renamed from R?; value R_US -> 3.3k; footprint (none) -> Resistor_SMD:R_1206_3216Metric
Connections:
- net labels added: +3.3V, A0, A1, Amp_Sensor, Vol_Sensor
- wire segments 14 -> 47
Other:
- moved on the sheet: C1, R1, R2
